Commit message: Tuning details of the gazebo simulation model.
1. Adjustments to inertials and dynamics settings to stabilise the simulation.
2. The ODE settings for cfm and erp are critical for a stable solution with this many constrained joints.

File: curio_description/urdf/curio.urdf.xacro (robot description, xacro)
@@ -77,5 +77,5 @@
     <xacro:property name="body_box_width" value="0.285" />
     <xacro:property name="body_box_depth" value="0.093" />
-    <xacro:property name="body_box_mass" value="0.500" />
+    <xacro:property name="body_box_mass" value="1.0" />
     <xacro:property name="front_rocker_arm_length" value="0.182" />
     <xacro:property name="back_rocker_arm_length" value="0.161" />
@@ -93,5 +93,5 @@
             <origin rpy="0 0 0" xyz="0 0 0" />
             <geometry>
-                <box size="0.001 0.001 0.001"/>
+                <box size="0.01 0.01 0.01"/>
             </geometry>
             <material name="orange" />
@@ -100,11 +100,11 @@
             <origin rpy="0 0 0" xyz="0 0 0" />
             <geometry>
-                <box size="0.001 0.001 0.001"/>
+                <box size="0.01 0.01 0.01"/>
             </geometry>
         </collision>
-        <inertial>
-            <mass value="0.01"/>
-            <inertia ixx="0.01" ixy="0" ixz="0" iyy="0.01" iyz="0" izz="0.01"/>
-        </inertial>
+        <xacro:solid_cuboid_inertial
+            rpy="0 0 0" xyz="0 0 0"
+            mass="0.01"
+            x="0.01" y="0.01" z="0.01" />
     </link>
     <gazebo reference="base_link">
@@ -139,6 +139,6 @@
     </joint>
     <gazebo reference="body_box_joint">
-        <disableFixedJointLumping>true</disableFixedJointLumping>
-        <preserveFixedJoint>true</preserveFixedJoint>
+        <!-- <disableFixedJointLumping>true</disableFixedJointLumping>  -->
+        <!-- <preserveFixedJoint>true</preserveFixedJoint> -->
     </gazebo>
     <!-- Differential
@@ -169,7 +169,12 @@
         <material>Gazebo/DarkGray</material>
     </gazebo>
-    <joint name="diff_brace_joint" type="continuous">
+    <joint name="diff_brace_joint" type="revolute">
         <origin rpy="0 0 0" xyz="0 0 0.0681"/>
         <axis xyz="0 0 1" />
+        <limit
+            lower="${-math_pi_over_4}"
+            upper="${math_pi_over_4}"
+            effort="100.0"
+            velocity="100.0" />
         <parent link="base_link" />
         <child link="diff_brace_link" />
@@ -178,6 +183,6 @@
         <provideFeedback>true</provideFeedback>
         <implicitSpringDamper>true</implicitSpringDamper>
-        <springStiffness>100.0</springStiffness>
-        <springReference>0.0</springReference>
+        <!-- <springStiffness>100.0</springStiffness> -->
+        <!-- <springReference>0.0</springReference> -->
     </gazebo>
     <!-- Turnbuckles -->
@@ -264,6 +269,11 @@
     <xacro:macro name="back_turnbuckle_socket_joint" params="lat_label reflect">
         <joint name="back_${lat_label}_turnbuckle_socket_joint" type="continuous">
-            <origin rpy="0 0 0" xyz="0 ${reflect * 0.16} 0"/>
+            <origin rpy="0 0 0" xyz="0 ${reflect * 0.17} 0"/>
             <axis xyz="0 1 0" />
+            <limit
+                lower="${-math_pi_over_4}"
+                upper="${math_pi_over_4}"
+                effort="100.0"
+                velocity="100.0" />
             <parent link="diff_brace_link" />
             <child link="back_${lat_label}_turnbuckle_socket_link" />
@@ -272,6 +282,6 @@
             <provideFeedback>true</provideFeedback>
             <implicitSpringDamper>true</implicitSpringDamper>
-            <springStiffness>100.0</springStiffness>
-            <springReference>0.0</springReference>
+            <!-- <springStiffness>100.0</springStiffness> -->
+            <!-- <springReference>0.0</springReference> -->
         </gazebo>
     </xacro:macro>
@@ -282,4 +292,9 @@
             <origin rpy="0 0 0" xyz="0 0 0"/>
             <axis xyz="0 0 1" />
+            <limit
+                lower="${-math_pi_over_4}"
+                upper="${math_pi_over_4}"
+                effort="100.0"
+                velocity="100.0" />
             <parent link="back_${lat_label}_turnbuckle_socket_link" />
             <child link="back_${lat_label}_turnbuckle_link" />
@@ -288,6 +303,6 @@
             <provideFeedback>true</provideFeedback>
             <implicitSpringDamper>true</implicitSpringDamper>
-            <springStiffness>100.0</springStiffness>
-            <springReference>0.0</springReference>
+            <!-- <springStiffness>100.0</springStiffness> -->
+            <!-- <springReference>0.0</springReference> -->
         </gazebo>
     </xacro:macro>
@@ -298,4 +313,9 @@
             <origin rpy="0 0 0" xyz="0 0 0"/>
             <axis xyz="0 1 0" />
+            <limit
+                lower="${-math_pi_over_4}"
+                upper="${math_pi_over_4}"
+                effort="100.0"
+                velocity="100.0" />
             <parent link="front_${lat_label}_turnbuckle_socket_link" />
             <child link="front_${lat_label}_turnbuckle_link" />
@@ -304,4 +324,6 @@
             <provideFeedback>true</provideFeedback>
             <implicitSpringDamper>true</implicitSpringDamper>
+            <!-- <springStiffness>100.0</springStiffness> -->
+            <!-- <springReference>0.0</springReference> -->
         </gazebo>
     </xacro:macro>
@@ -310,6 +332,11 @@
     <xacro:macro name="front_turnbuckle_socket_joint" params="lat_label reflect">
         <joint name="front_${lat_label}_turnbuckle_socket_joint" type="continuous">
-            <origin rpy="0 0 0" xyz="0 0 0.07"/>
+            <origin rpy="0 0 0" xyz="0 ${reflect * 0.02} 0.0565"/>
             <axis xyz="0 0 1" />
+            <limit
+                lower="${-math_pi_over_4}"
+                upper="${math_pi_over_4}"
+                effort="100.0"
+                velocity="100.0" />
             <parent link="${lat_label}_rocker_link" />
             <child link="front_${lat_label}_turnbuckle_socket_link" />
@@ -318,11 +345,11 @@
             <provideFeedback>true</provideFeedback>
             <implicitSpringDamper>true</implicitSpringDamper>
-            <springStiffness>100.0</springStiffness>
-            <springReference>0.0</springReference>
+            <!-- <springStiffness>100.0</springStiffness> -->
+            <!-- <springReference>0.0</springReference> -->
         </gazebo>
     </xacro:macro>
     <xacro:front_turnbuckle_socket_joint lat_label="left" reflect="1"/>
     <xacro:front_turnbuckle_socket_joint lat_label="right" reflect="-1"/>
-    <!-- Gazebo only fixed link to close differential linkage loop -->
+    <!-- Gazebo only §link to close differential linkage loop -->
     <gazebo>
         <joint name="left_turnbuckle_joint" type="revolute">
@@ -333,8 +360,4 @@
             <parent>back_left_turnbuckle_link</parent>
             <child>front_left_turnbuckle_link</child>
-            <dynamics>
-                <spring_stiffness>100.0</spring_stiffness>
-                <spring_reference>0</spring_reference>
-            </dynamics>
             <physics>
                 <ode>
@@ -350,8 +373,4 @@
             <parent>back_right_turnbuckle_link</parent>
             <child>front_right_turnbuckle_link</child>
-            <dynamics>
-                <spring_stiffness>100.0</spring_stiffness>
-                <spring_reference>0</spring_reference>
-            </dynamics>
             <physics>
                 <ode>
@@ -379,5 +398,5 @@
             <xacro:solid_cuboid_inertial
                 rpy="0 0 0" xyz="0 0 0"
-                mass="0.1"
+                mass="0.25"
                 x="0.1" y="0.015" z="0.015" />
         </link>
@@ -388,8 +407,14 @@
     <xacro:rocker_link lat_label="left" reflect="1"/>
     <xacro:rocker_link lat_label="right" reflect="-1"/>
+    <!-- Continuous Rocker Joint  -->
     <xacro:macro name="rocker_joint" params="lat_label reflect">
         <joint name="${lat_label}_rocker_joint" type="continuous">
-            <origin rpy="0 0 0" xyz="0.071 ${reflect * 0.154} 0.0118"/>
+            <origin rpy="0 0 0" xyz="0.071 ${reflect * 0.15} 0.0118"/>
             <axis xyz="0 1 0" />
+            <limit
+                lower="${-math_pi_over_4}"
+                upper="${math_pi_over_4}"
+                effort="100.0"
+                velocity="100.0" />
             <parent link="base_link" />
             <child link="${lat_label}_rocker_link" />
@@ -397,9 +422,21 @@
         <gazebo reference="${lat_label}_rocker_joint">
             <provideFeedback>true</provideFeedback>
-            <!-- <implicitSpringDamper>true</implicitSpringDamper>
-            <springStiffness>0.0</springStiffness>
-            <springReference>0.0</springReference> -->
-        </gazebo>
-    </xacro:macro>
+            <implicitSpringDamper>true</implicitSpringDamper>
+            <!-- <springStiffness>100.0</springStiffness> -->
+            <!-- <springReference>0.0</springReference> -->
+        </gazebo>
+    </xacro:macro>
+    <!-- Fixed Rocker Joint  -->
+    <!-- <xacro:macro name="rocker_joint" params="lat_label reflect">
+        <joint name="${lat_label}_rocker_joint" type="fixed">
+            <origin rpy="0 0 0" xyz="0.071 ${reflect * 0.154} 0.0118"/>
+            <parent link="base_link" />
+            <child link="${lat_label}_rocker_link" />
+        </joint>
+        <gazebo reference="${lat_label}_rocker_joint">
+            <disableFixedJointLumping>true</disableFixedJointLumping>
+            <preserveFixedJoint>true</preserveFixedJoint>
+        </gazebo>
+    </xacro:macro> -->
     <xacro:rocker_joint lat_label="left" reflect="1"/>
     <xacro:rocker_joint lat_label="right" reflect="-1"/>
@@ -421,5 +458,5 @@
             <xacro:solid_cuboid_inertial
                 rpy="0 0 0" xyz="0 0 0"
-                mass="0.1"
+                mass="0.25"
                 x="0.1" y="0.1" z="0.1" />
         </link>
@@ -439,6 +476,6 @@
         <gazebo reference="front_${lat_label}_corner_joint">
             <provideFeedback>true</provideFeedback>
-            <!-- <implicitSpringDamper>true</implicitSpringDamper>
-            <springStiffness>0.0</springStiffness>
+            <implicitSpringDamper>true</implicitSpringDamper>
+            <!-- <springStiffness>0.0</springStiffness>
             <springReference>0.0</springReference> -->
         </gazebo>
@@ -463,5 +500,5 @@
             <xacro:solid_cylinder_inertial
                 rpy="0 0 0" xyz="0 0 0"
-                mass="0.1"
+                mass="0.25"
                 radius="${wheel_radius}" length="${wheel_width}" />
         </link>
@@ -481,7 +518,7 @@
         <gazebo reference="${lon_label}_${lat_label}_wheel_joint">
             <provideFeedback>true</provideFeedback>
-            <!-- <implicitSpringDamper>true</implicitSpringDamper>
-            <springStiffness>0.0</springStiffness>
-            <springReference>0.0</springReference> -->
+            <implicitSpringDamper>true</implicitSpringDamper>
+            <!-- <springStiffness>0.0</springStiffness> -->
+            <!-- <springReference>0.0</springReference> -->
         </gazebo>
     </xacro:macro>
@@ -506,5 +543,5 @@
             <xacro:solid_cuboid_inertial
                 rpy="0 0 0" xyz="0 0 0"
-                mass="0.1"
+                mass="0.25"
                 x="0.1" y="0.015" z="0.015" />
         </link>
@@ -515,8 +552,14 @@
     <xacro:bogie_link lat_label="left" reflect="1"/>
     <xacro:bogie_link lat_label="right" reflect="-1"/>
+    <!-- Continuous Bogie Joint  -->
     <xacro:macro name="bogie_joint" params="lat_label reflect">
-        <joint name="${lat_label}_bogie_joint" type="continuous">
+        <joint name="${lat_label}_bogie_joint" type="revolute">
             <origin rpy="0 0 0" xyz="-0.181 ${reflect * 0.0675} -0.062"/>
             <axis xyz="0 1 0" />
+            <limit
+                lower="${-math_pi_over_4}"
+                upper="${math_pi_over_4}"
+                effort="100.0"
+                velocity="100.0" />
             <parent link="${lat_label}_rocker_link" />
             <child link="${lat_label}_bogie_link" />
@@ -524,9 +567,21 @@
         <gazebo reference="${lat_label}_bogie_joint">
             <provideFeedback>true</provideFeedback>
-            <!-- <implicitSpringDamper>true</implicitSpringDamper>
-            <springStiffness>0.0</springStiffness>
-            <springReference>0.0</springReference> -->
-        </gazebo>
-    </xacro:macro>
+            <implicitSpringDamper>true</implicitSpringDamper>
+            <!-- <springStiffness>0.0</springStiffness> -->
+            <!-- <springReference>0.0</springReference> -->
+        </gazebo>
+    </xacro:macro>
+    <!-- Fixed Bogie Joint  -->
+    <!-- <xacro:macro name="bogie_joint" params="lat_label reflect">
+        <joint name="${lat_label}_bogie_joint" type="fixed">
+            <origin rpy="0 0 0" xyz="-0.181 ${reflect * 0.0675} -0.062"/>
+            <parent link="${lat_label}_rocker_link" />
+            <child link="${lat_label}_bogie_link" />
+        </joint>
+        <gazebo reference="${lat_label}_bogie_joint">
+            <disableFixedJointLumping>true</disableFixedJointLumping>
+            <preserveFixedJoint>true</preserveFixedJoint>
+        </gazebo>
+    </xacro:macro> -->
     <xacro:bogie_joint lat_label="left" reflect="1"/>
     <xacro:bogie_joint lat_label="right" reflect="-1"/>
@@ -542,7 +597,7 @@
         <gazebo reference="mid_${lat_label}_wheel_joint">
             <provideFeedback>true</provideFeedback>
-            <!-- <implicitSpringDamper>true</implicitSpringDamper>
-            <springStiffness>0.0</springStiffness>
-            <springReference>0.0</springReference> -->
+            <implicitSpringDamper>true</implicitSpringDamper>
+            <!-- <springStiffness>0.0</springStiffness> -->
+            <!-- <springReference>0.0</springReference> -->
         </gazebo>
     </xacro:macro>
@@ -560,7 +615,7 @@
         <gazebo reference="back_${lat_label}_corner_joint">
             <provideFeedback>true</provideFeedback>
-            <!-- <implicitSpringDamper>true</implicitSpringDamper>
-            <springStiffness>0.0</springStiffness>
-            <springReference>0.0</springReference> -->
+            <implicitSpringDamper>true</implicitSpringDamper>
+            <!-- <springStiffness>0.0</springStiffness> -->
+            <!-- <springReference>0.0</springReference> -->
         </gazebo>
     </xacro:macro>

Commit message: Improvements to the robot description. Add mesh files.
1. Second draft of model description using exported STL files.

File: curio_description/urdf/curio.urdf.xacro (robot description, xacro)
@@ -49,4 +49,6 @@
             Resources:
                 http://answers.gazebosim.org/question/13844/getting-joint-angles-for-passive-urdf-model/
+            Gazebo only joints
+                left_turnbuckle_joint, right_turnbuckle_joint
          -->
         <plugin name="gazebo_ros_joint_state_publisher" filename="libgazebo_ros_joint_state_publisher.so">
@@ -63,6 +65,5 @@
                 back_left_turnbuckle_joint, back_right_turnbuckle_joint,
                 front_left_turnbuckle_socket_joint, front_right_turnbuckle_socket_joint,
-                front_left_turnbuckle_joint, front_right_turnbuckle_joint,
-                left_turnbuckle_joint, right_turnbuckle_joint
+                front_left_turnbuckle_joint, front_right_turnbuckle_joint
             </jointName>
             <updateRate>50</updateRate>
@@ -115,5 +116,6 @@
             <origin rpy="0 0 0" xyz="0 0 0" />
             <geometry>
-                <box size="${body_box_length} ${body_box_width} ${body_box_depth}"/>
+                <mesh filename="package://curio_description/meshes/bases/body_box.stl" />
+                <!-- <box size="${body_box_length} ${body_box_width} ${body_box_depth}"/> -->
             </geometry>
             <material name="dark_gray" />
@@ -149,7 +151,9 @@
     <link name="diff_brace_link">
         <visual>
-            <origin rpy="0 0 ${math_pi_over_2}" xyz="0 0 0" />
+            <origin rpy="0 0 0" xyz="0 0 0" />
+            <!-- <origin rpy="0 0 ${math_pi_over_2}" xyz="0 0 0" /> -->
             <geometry>
-                <box size="0.200 0.015 0.015"/>
+                <mesh filename="package://curio_description/meshes/bases/differential.stl" />
+                <!-- <box size="0.200 0.015 0.015"/> -->
             </geometry>
             <material name="dark_gray" />
@@ -192,5 +196,5 @@
                 <origin rpy="0 0 0" xyz="0 0 0" />
                 <geometry>
-                    <box size="0.005 0.005 0.005"/>
+                    <sphere radius="0.0025"/>
                 </geometry>
                 <material name="dark_gray" />
@@ -199,5 +203,5 @@
                 <origin rpy="0 0 0" xyz="0 0 0" />
                 <geometry>
-                    <box size="0.005 0.005 0.005"/>
+                    <sphere radius="0.0025"/>
                 </geometry>
             </collision>
@@ -218,20 +222,20 @@
         <link name="back_${lat_label}_turnbuckle_link">
             <visual>
-                <origin rpy="0 0 0" xyz="0.02 0 0" />
-                <geometry>
-                    <box size="0.04 0.005 0.005"/>
+                <origin rpy="0 ${math_pi_over_2} 0" xyz="0.02 0 0" />
+                <geometry>
+                    <cylinder length="0.04" radius="0.0025" />
                 </geometry>
                 <material name="dark_gray" />
             </visual>
             <collision>
-                <origin rpy="0 0 0" xyz="0 0 0" />
-                <geometry>
-                    <box size="0.04 0.005 0.005"/>
+                <origin rpy="0 ${math_pi_over_2} 0" xyz="0.02 0 0" />
+                <geometry>
+                    <cylinder length="0.04" radius="0.0025" />
                 </geometry>
             </collision>
-            <xacro:solid_cuboid_inertial
+            <xacro:solid_cylinder_inertial
                 rpy="0 0 0" xyz="0 0 0"
                 mass="0.01"
-                x="0.04" y="0.005" z="0.005" />
+                length="0.04" radius="0.0025" />
         </link>
         <gazebo reference="back_${lat_label}_turnbuckle_link">
@@ -244,20 +248,20 @@
         <link name="front_${lat_label}_turnbuckle_link">
             <visual>
-                <origin rpy="0 0 0" xyz="-0.02 0 0" />
-                <geometry>
-                    <box size="0.04 0.005 0.005"/>
+                <origin rpy="0 ${math_pi_over_2} 0" xyz="-0.015 0 0" />
+                <geometry>
+                    <cylinder length="0.03" radius="0.0025" />
                 </geometry>
                 <material name="dark_gray" />
             </visual>
             <collision>
-                <origin rpy="0 0 0" xyz="0 0 0" />
-                <geometry>
-                    <box size="0.04 0.005 0.005"/>
+                <origin rpy="0 ${math_pi_over_2} 0" xyz="-0.015 0 0" />
+                <geometry>
+                    <cylinder length="0.03" radius="0.0025" />
                 </geometry>
             </collision>
-            <xacro:solid_cuboid_inertial
+            <xacro:solid_cylinder_inertial
                 rpy="0 0 0" xyz="0 0 0"
                 mass="0.01"
-                x="0.04" y="0.005" z="0.005" />
+                length="0.03" radius="0.0025" />
         </link>
         <gazebo reference="front_${lat_label}_turnbuckle_link">
@@ -332,5 +336,5 @@
     <xacro:macro name="front_turnbuckle_socket_joint" params="lat_label reflect">
         <joint name="front_${lat_label}_turnbuckle_socket_joint" type="continuous">
-            <origin rpy="0 0 0" xyz="0 ${reflect * 0.02} 0.0565"/>
+            <origin rpy="0 0 0" xyz="0.0 ${reflect * 0.0146} 0.0565"/>
             <axis xyz="0 0 1" />
             <limit
@@ -354,5 +358,5 @@
     <gazebo>
         <joint name="left_turnbuckle_joint" type="revolute">
-            <pose>-0.04 0 0 0 0 0</pose>
+            <pose>-0.03 0 0 0 0 0</pose>
             <axis>
                 <xyz>1 0 0</xyz>
@@ -367,5 +371,5 @@
         </joint>
         <joint name="right_turnbuckle_joint" type="revolute">
-            <pose>-0.04 0 0 0 0 0</pose>
+            <pose>-0.03 0 0 0 0 0</pose>
             <axis>
                 <xyz>1 0 0</xyz>
@@ -386,5 +390,6 @@
                 <origin rpy="0 0 0" xyz="0 0 0" />
                 <geometry>
-                    <box size="0.1 0.015 0.015"/>
+                    <mesh filename="package://curio_description/meshes/bases/${lat_label}_rocker_asm.stl" />
+                    <!-- <box size="0.1 0.015 0.015"/> -->
                 </geometry>
                 <material name="dark_gray" />
@@ -410,5 +415,5 @@
     <xacro:macro name="rocker_joint" params="lat_label reflect">
         <joint name="${lat_label}_rocker_joint" type="continuous">
-            <origin rpy="0 0 0" xyz="0.071 ${reflect * 0.15} 0.0118"/>
+            <origin rpy="0 0 0" xyz="0.071 ${reflect * 0.155} 0.0118"/>
             <axis xyz="0 1 0" />
             <limit
@@ -446,5 +451,6 @@
                 <origin rpy="0 0 0" xyz="0 0 0" />
                 <geometry>
-                    <box size="0.1 0.1 0.1"/>
+                    <mesh filename="package://curio_description/meshes/bases/${lon_label}_${lat_label}_steering_asm.stl" />
+                    <!-- <box size="0.1 0.1 0.1"/> -->
                 </geometry>
                 <material name="dark_gray" />
@@ -469,5 +475,5 @@
     <xacro:macro name="front_corner_joint" params="lat_label reflect">
         <joint name="front_${lat_label}_corner_joint" type="continuous">
-            <origin rpy="0 0 0" xyz="0.2116 ${reflect * 0.081} -0.0279"/>
+            <origin rpy="0 0 0" xyz="0.2116 ${reflect * 0.075} -0.0279"/>
             <axis xyz="0 0 1" />
             <parent link="${lat_label}_rocker_link" />
@@ -531,5 +537,6 @@
                 <origin rpy="0 0 0" xyz="0 0 0" />
                 <geometry>
-                    <box size="0.1 0.015 0.015"/>
+                    <mesh filename="package://curio_description/meshes/bases/${lat_label}_bogie_asm.stl" />
+                    <!-- <box size="0.1 0.015 0.015"/> -->
                 </geometry>
                 <material name="dark_gray" />
@@ -555,5 +562,5 @@
     <xacro:macro name="bogie_joint" params="lat_label reflect">
         <joint name="${lat_label}_bogie_joint" type="revolute">
-            <origin rpy="0 0 0" xyz="-0.181 ${reflect * 0.0675} -0.062"/>
+            <origin rpy="0 0 0" xyz="-0.181 ${reflect * 0.025} -0.062"/>
             <axis xyz="0 1 0" />
             <limit
@@ -608,5 +615,5 @@
     <xacro:macro name="back_corner_joint" params="lat_label reflect">
         <joint name="back_${lat_label}_corner_joint" type="continuous">
-            <origin rpy="0 0 0" xyz="-0.149 ${reflect * 0.0136} 0.0338"/>
+            <origin rpy="0 0 0" xyz="-0.149 ${reflect * 0.05} 0.0338"/>
             <axis xyz="0 0 1" />
             <parent link="${lat_label}_bogie_link" />
