Commit message: Updates to robot meshes and further tuning of urdf model.
1. Add mesh for turnbuckle.
2. Correct orientation of steering assemblies
3. Remove duplicate wheel assemblies.

File: curio_description/urdf/curio.urdf.xacro (robot description, xacro)
@@ -222,9 +222,12 @@
         <link name="back_${lat_label}_turnbuckle_link">
             <visual>
-                <origin rpy="0 ${math_pi_over_2} 0" xyz="0.02 0 0" />
-                <geometry>
-                    <cylinder length="0.04" radius="0.0025" />
-                </geometry>
-                <material name="dark_gray" />
+                <!-- <origin rpy="0 -0.1 ${-reflect * 0.15}" xyz="0.037 ${-reflect * 0.005} 0.002" /> -->
+                <origin rpy="0 0 0" xyz="0.035 0 0" />
+                <!-- <origin rpy="0 ${math_pi_over_2} 0" xyz="0.02 0 0" /> -->
+                <geometry>
+                    <mesh filename="package://curio_description/meshes/bases/turnbuckle.stl" />
+                    <!-- <cylinder length="0.04" radius="0.0025" /> -->
+                </geometry>
+                <material name="blue" />
             </visual>
             <collision>
@@ -247,5 +250,5 @@
     <xacro:macro name="front_turnbuckle_link" params="lat_label reflect">
         <link name="front_${lat_label}_turnbuckle_link">
-            <visual>
+            <!-- <visual>
                 <origin rpy="0 ${math_pi_over_2} 0" xyz="-0.015 0 0" />
                 <geometry>
@@ -253,5 +256,5 @@
                 </geometry>
                 <material name="dark_gray" />
-            </visual>
+            </visual> -->
             <collision>
                 <origin rpy="0 ${math_pi_over_2} 0" xyz="-0.015 0 0" />
@@ -355,5 +358,5 @@
     <xacro:front_turnbuckle_socket_joint lat_label="left" reflect="1"/>
     <xacro:front_turnbuckle_socket_joint lat_label="right" reflect="-1"/>
-    <!-- Gazebo only §link to close differential linkage loop -->
+    <!-- Gazebo only link to close differential linkage loop -->
     <gazebo>
         <joint name="left_turnbuckle_joint" type="revolute">
@@ -494,5 +497,5 @@
                 <origin rpy="${reflect * math_pi_over_2} 0 0" xyz="0 0 0" />
                 <geometry>
-                    <mesh filename="package://curio_description/meshes/wheels/wheel.stl" />
+                    <mesh filename="package://curio_description/meshes/wheels/wheel_asm.stl" />
                 </geometry>
                 <material name="dark_gray" />

Commit message: Add package for a controller using the ros_control framework.
1. This version implements a diff_drive_controller using the ros_controllers code (to establish the package and plugin mechanisms work).

File: curio_description/urdf/curio.urdf.xacro (robot description, xacro)
@@ -49,4 +49,8 @@
             Resources:
                 http://answers.gazebosim.org/question/13844/getting-joint-angles-for-passive-urdf-model/
+            Wheel joints controlled by the diff_drive_controller
+                front_left_wheel_joint, front_right_wheel_joint,
+                mid_left_wheel_joint, mid_right_wheel_joint,
+                back_left_wheel_joint, back_right_wheel_joint,
             Gazebo only joints
                 left_turnbuckle_joint, right_turnbuckle_joint
@@ -56,14 +60,12 @@
             <jointName>
                 left_rocker_joint, right_rocker_joint,
+                left_bogie_joint, right_bogie_joint,
                 front_left_corner_joint, front_right_corner_joint,
-                front_left_wheel_joint, front_right_wheel_joint,
-                left_bogie_joint, right_bogie_joint,
-                mid_left_wheel_joint, mid_right_wheel_joint,
                 back_left_corner_joint, back_right_corner_joint,
-                back_left_wheel_joint, back_right_wheel_joint,
                 back_left_turnbuckle_socket_joint, back_right_turnbuckle_socket_joint,
                 back_left_turnbuckle_joint, back_right_turnbuckle_joint,
                 front_left_turnbuckle_socket_joint, front_right_turnbuckle_socket_joint,
-                front_left_turnbuckle_joint, front_right_turnbuckle_joint
+                front_left_turnbuckle_joint, front_right_turnbuckle_joint,
+                left_turnbuckle_joint, right_turnbuckle_joint
             </jointName>
             <updateRate>50</updateRate>
@@ -483,9 +485,15 @@
             <child link="front_${lat_label}_corner_link" />
         </joint>
+        <transmission name="front_${lat_label}_corner_transmission" >
+            <type>transmission_interface/SimpleTransmission</type>
+            <actuator name="front_${lat_label}_corner_actuator">
+                <mechanicalReduction>1</mechanicalReduction>
+            </actuator>
+            <joint name="front_${lat_label}_corner_joint">
+                <hardwareInterface>hardware_interface/PositionJointInterface</hardwareInterface>
+            </joint>
+        </transmission>
         <gazebo reference="front_${lat_label}_corner_joint">
             <provideFeedback>true</provideFeedback>
-            <implicitSpringDamper>true</implicitSpringDamper>
-            <!-- <springStiffness>0.0</springStiffness>
-            <springReference>0.0</springReference> -->
         </gazebo>
     </xacro:macro>
@@ -525,9 +533,15 @@
             <child link="${lon_label}_${lat_label}_wheel_link" />
         </joint>
+        <transmission name="${lon_label}_${lat_label}_wheel_transmission" >
+            <type>transmission_interface/SimpleTransmission</type>
+            <actuator name="${lon_label}_${lat_label}_wheel_actuator">
+                <mechanicalReduction>1</mechanicalReduction>
+            </actuator>
+            <joint name="${lon_label}_${lat_label}_wheel_joint">
+                <hardwareInterface>hardware_interface/VelocityJointInterface</hardwareInterface>
+            </joint>
+        </transmission>
         <gazebo reference="${lon_label}_${lat_label}_wheel_joint">
             <provideFeedback>true</provideFeedback>
-            <implicitSpringDamper>true</implicitSpringDamper>
-            <!-- <springStiffness>0.0</springStiffness> -->
-            <!-- <springReference>0.0</springReference> -->
         </gazebo>
     </xacro:macro>
@@ -605,9 +619,15 @@
             <child link="mid_${lat_label}_wheel_link" />
         </joint>
+        <transmission name="mid_${lat_label}_wheel_transmission" >
+            <type>transmission_interface/SimpleTransmission</type>
+            <actuator name="mid_${lat_label}_wheel_actuator">
+                <mechanicalReduction>1</mechanicalReduction>
+            </actuator>
+            <joint name="mid_${lat_label}_wheel_joint">
+                <hardwareInterface>hardware_interface/VelocityJointInterface</hardwareInterface>
+            </joint>
+        </transmission>
         <gazebo reference="mid_${lat_label}_wheel_joint">
             <provideFeedback>true</provideFeedback>
-            <implicitSpringDamper>true</implicitSpringDamper>
-            <!-- <springStiffness>0.0</springStiffness> -->
-            <!-- <springReference>0.0</springReference> -->
         </gazebo>
     </xacro:macro>
@@ -623,9 +643,15 @@
             <child link="back_${lat_label}_corner_link" />
         </joint>
+        <transmission name="back_${lat_label}_corner_transmission" >
+            <type>transmission_interface/SimpleTransmission</type>
+            <actuator name="back_${lat_label}_corner_actuator">
+                <mechanicalReduction>1</mechanicalReduction>
+            </actuator>
+            <joint name="back_${lat_label}_corner_joint">
+                <hardwareInterface>hardware_interface/PositionJointInterface</hardwareInterface>
+            </joint>
+        </transmission>
         <gazebo reference="back_${lat_label}_corner_joint">
             <provideFeedback>true</provideFeedback>
-            <implicitSpringDamper>true</implicitSpringDamper>
-            <!-- <springStiffness>0.0</springStiffness> -->
-            <!-- <springReference>0.0</springReference> -->
         </gazebo>
     </xacro:macro>
