Commit message: Change implementation of turnbuckle linkages to gazebo links and ball joints.
1. The original turnbuckle linkages were too complicated and seemed to 'separate' in simulation leading to the body being unsupported. This change fixes that.

File: curio_description/urdf/curio.urdf.xacro (robot description, xacro)
@@ -49,23 +49,24 @@
             Resources:
                 http://answers.gazebosim.org/question/13844/getting-joint-angles-for-passive-urdf-model/
-            Wheel joints controlled by the diff_drive_controller
+            Wheel joints controlled by ros_control diff_drive_controller:
                 front_left_wheel_joint, front_right_wheel_joint,
                 mid_left_wheel_joint, mid_right_wheel_joint,
-                back_left_wheel_joint, back_right_wheel_joint,
-            Gazebo only joints
-                left_turnbuckle_joint, right_turnbuckle_joint
+                back_left_wheel_joint, back_right_wheel_joint
+            Gazebo only links:
+                left_turnbuckle_link, right_turnbuckle_link
+            Gazebo only joints:
+                back_left_turnbuckle_joint, back_right_turnbuckle_joint,
+                front_left_turnbuckle_joint, front_right_turnbuckle_joint
          -->
         <plugin name="gazebo_ros_joint_state_publisher" filename="libgazebo_ros_joint_state_publisher.so">
             <robotNamespace>/</robotNamespace>
             <jointName>
+                front_left_corner_joint, front_right_corner_joint,
+                back_left_corner_joint, back_right_corner_joint,
                 left_rocker_joint, right_rocker_joint,
                 left_bogie_joint, right_bogie_joint,
-                front_left_corner_joint, front_right_corner_joint,
-                back_left_corner_joint, back_right_corner_joint,
-                back_left_turnbuckle_socket_joint, back_right_turnbuckle_socket_joint,
+                diff_brace_joint,
                 back_left_turnbuckle_joint, back_right_turnbuckle_joint,
-                front_left_turnbuckle_socket_joint, front_right_turnbuckle_socket_joint,
-                front_left_turnbuckle_joint, front_right_turnbuckle_joint,
-                left_turnbuckle_joint, right_turnbuckle_joint
+                front_left_turnbuckle_joint, front_right_turnbuckle_joint
             </jointName>
             <updateRate>50</updateRate>
@@ -146,9 +147,5 @@
         <!-- <preserveFixedJoint>true</preserveFixedJoint> -->
     </gazebo>
-    <!-- Differential
-        TODO: Implementing the differential is tricky
-        URDF does not support closed loops in the robot description,
-        on the other hand SDF for Gazebo does.
-    -->
+    <!-- Differential -->
     <link name="diff_brace_link">
         <visual>
@@ -192,201 +189,66 @@
         <!-- <springReference>0.0</springReference> -->
     </gazebo>
-    <!-- Turnbuckles -->
-    <xacro:macro name="turnbuckle_socket_link" params="lon_label lat_label reflect">
-        <link name="${lon_label}_${lat_label}_turnbuckle_socket_link">
-            <visual>
-                <origin rpy="0 0 0" xyz="0 0 0" />
-                <geometry>
-                    <sphere radius="0.0025"/>
-                </geometry>
-                <material name="dark_gray" />
-            </visual>
-            <collision>
-                <origin rpy="0 0 0" xyz="0 0 0" />
-                <geometry>
-                    <sphere radius="0.0025"/>
-                </geometry>
-            </collision>
-            <xacro:solid_cuboid_inertial
-                rpy="0 0 0" xyz="0 0 0"
-                mass="0.01"
-                x="0.005" y="0.005" z="0.005" />
-        </link>
-        <gazebo reference="${lon_label}_${lat_label}_turnbuckle_socket_link">
-            <material>Gazebo/Red</material>
-        </gazebo>
-    </xacro:macro>
-    <xacro:turnbuckle_socket_link lon_label="back" lat_label="left" reflect="1"/>
-    <xacro:turnbuckle_socket_link lon_label="back" lat_label="right" reflect="-1"/>
-    <xacro:turnbuckle_socket_link lon_label="front" lat_label="left" reflect="1"/>
-    <xacro:turnbuckle_socket_link lon_label="front" lat_label="right" reflect="-1"/>
-    <xacro:macro name="back_turnbuckle_link" params="lat_label reflect">
-        <link name="back_${lat_label}_turnbuckle_link">
-            <visual>
-                <!-- <origin rpy="0 -0.1 ${-reflect * 0.15}" xyz="0.037 ${-reflect * 0.005} 0.002" /> -->
-                <origin rpy="0 0 0" xyz="0.035 0 0" />
-                <!-- <origin rpy="0 ${math_pi_over_2} 0" xyz="0.02 0 0" /> -->
-                <geometry>
-                    <mesh filename="package://curio_description/meshes/bases/turnbuckle.stl" />
-                    <!-- <cylinder length="0.04" radius="0.0025" /> -->
-                </geometry>
-                <material name="blue" />
-            </visual>
-            <collision>
-                <origin rpy="0 ${math_pi_over_2} 0" xyz="0.02 0 0" />
-                <geometry>
-                    <cylinder length="0.04" radius="0.0025" />
-                </geometry>
-            </collision>
-            <xacro:solid_cylinder_inertial
-                rpy="0 0 0" xyz="0 0 0"
-                mass="0.01"
-                length="0.04" radius="0.0025" />
-        </link>
-        <gazebo reference="back_${lat_label}_turnbuckle_link">
-            <material>Gazebo/Blue</material>
-        </gazebo>
-    </xacro:macro>
-    <xacro:back_turnbuckle_link lat_label="left" reflect="1"/>
-    <xacro:back_turnbuckle_link lat_label="right" reflect="-1"/>
-    <xacro:macro name="front_turnbuckle_link" params="lat_label reflect">
-        <link name="front_${lat_label}_turnbuckle_link">
-            <!-- <visual>
-                <origin rpy="0 ${math_pi_over_2} 0" xyz="-0.015 0 0" />
-                <geometry>
-                    <cylinder length="0.03" radius="0.0025" />
-                </geometry>
-                <material name="dark_gray" />
-            </visual> -->
-            <collision>
-                <origin rpy="0 ${math_pi_over_2} 0" xyz="-0.015 0 0" />
-                <geometry>
-                    <cylinder length="0.03" radius="0.0025" />
-                </geometry>
-            </collision>
-            <xacro:solid_cylinder_inertial
-                rpy="0 0 0" xyz="0 0 0"
-                mass="0.01"
-                length="0.03" radius="0.0025" />
-        </link>
-        <gazebo reference="front_${lat_label}_turnbuckle_link">
-            <material>Gazebo/Blue</material>
-        </gazebo>
-    </xacro:macro>
-    <xacro:front_turnbuckle_link lat_label="left" reflect="1"/>
-    <xacro:front_turnbuckle_link lat_label="right" reflect="-1"/>
-    <xacro:macro name="back_turnbuckle_socket_joint" params="lat_label reflect">
-        <joint name="back_${lat_label}_turnbuckle_socket_joint" type="continuous">
-            <origin rpy="0 0 0" xyz="0 ${reflect * 0.17} 0"/>
-            <axis xyz="0 1 0" />
-            <limit
-                lower="${-math_pi_over_4}"
-                upper="${math_pi_over_4}"
-                effort="100.0"
-                velocity="100.0" />
-            <parent link="diff_brace_link" />
-            <child link="back_${lat_label}_turnbuckle_socket_link" />
-        </joint>
-        <gazebo reference="back_${lat_label}_turnbuckle_socket_joint">
-            <provideFeedback>true</provideFeedback>
-            <implicitSpringDamper>true</implicitSpringDamper>
-            <!-- <springStiffness>100.0</springStiffness> -->
-            <!-- <springReference>0.0</springReference> -->
-        </gazebo>
-    </xacro:macro>
-    <xacro:back_turnbuckle_socket_joint lat_label="left" reflect="1"/>
-    <xacro:back_turnbuckle_socket_joint lat_label="right" reflect="-1"/>
-    <xacro:macro name="back_turnbuckle_joint" params="lat_label reflect">
-        <joint name="back_${lat_label}_turnbuckle_joint" type="continuous">
-            <origin rpy="0 0 0" xyz="0 0 0"/>
-            <axis xyz="0 0 1" />
-            <limit
-                lower="${-math_pi_over_4}"
-                upper="${math_pi_over_4}"
-                effort="100.0"
-                velocity="100.0" />
-            <parent link="back_${lat_label}_turnbuckle_socket_link" />
-            <child link="back_${lat_label}_turnbuckle_link" />
-        </joint>
-        <gazebo reference="back_${lat_label}_turnbuckle_joint">
-            <provideFeedback>true</provideFeedback>
-            <implicitSpringDamper>true</implicitSpringDamper>
-            <!-- <springStiffness>100.0</springStiffness> -->
-            <!-- <springReference>0.0</springReference> -->
-        </gazebo>
-    </xacro:macro>
-    <xacro:back_turnbuckle_joint lat_label="left" reflect="1"/>
-    <xacro:back_turnbuckle_joint lat_label="right" reflect="-1"/>
-    <xacro:macro name="front_turnbuckle_joint" params="lat_label reflect">
-        <joint name="front_${lat_label}_turnbuckle_joint" type="continuous">
-            <origin rpy="0 0 0" xyz="0 0 0"/>
-            <axis xyz="0 1 0" />
-            <limit
-                lower="${-math_pi_over_4}"
-                upper="${math_pi_over_4}"
-                effort="100.0"
-                velocity="100.0" />
-            <parent link="front_${lat_label}_turnbuckle_socket_link" />
-            <child link="front_${lat_label}_turnbuckle_link" />
-        </joint>
-        <gazebo reference="front_${lat_label}_turnbuckle_joint">
-            <provideFeedback>true</provideFeedback>
-            <implicitSpringDamper>true</implicitSpringDamper>
-            <!-- <springStiffness>100.0</springStiffness> -->
-            <!-- <springReference>0.0</springReference> -->
-        </gazebo>
-    </xacro:macro>
-    <xacro:front_turnbuckle_joint lat_label="left" reflect="1"/>
-    <xacro:front_turnbuckle_joint lat_label="right" reflect="-1"/>
-    <xacro:macro name="front_turnbuckle_socket_joint" params="lat_label reflect">
-        <joint name="front_${lat_label}_turnbuckle_socket_joint" type="continuous">
-            <origin rpy="0 0 0" xyz="0.0 ${reflect * 0.0146} 0.0565"/>
-            <axis xyz="0 0 1" />
-            <limit
-                lower="${-math_pi_over_4}"
-                upper="${math_pi_over_4}"
-                effort="100.0"
-                velocity="100.0" />
-            <parent link="${lat_label}_rocker_link" />
-            <child link="front_${lat_label}_turnbuckle_socket_link" />
-        </joint>
-        <gazebo reference="front_${lat_label}_turnbuckle_joint">
-            <provideFeedback>true</provideFeedback>
-            <implicitSpringDamper>true</implicitSpringDamper>
-            <!-- <springStiffness>100.0</springStiffness> -->
-            <!-- <springReference>0.0</springReference> -->
-        </gazebo>
-    </xacro:macro>
-    <xacro:front_turnbuckle_socket_joint lat_label="left" reflect="1"/>
-    <xacro:front_turnbuckle_socket_joint lat_label="right" reflect="-1"/>
-    <!-- Gazebo only link to close differential linkage loop -->
-    <gazebo>
-        <joint name="left_turnbuckle_joint" type="revolute">
-            <pose>-0.03 0 0 0 0 0</pose>
-            <axis>
-                <xyz>1 0 0</xyz>
-            </axis>
-            <parent>back_left_turnbuckle_link</parent>
-            <child>front_left_turnbuckle_link</child>
-            <physics>
-                <ode>
-                    <implicit_spring_damper>1</implicit_spring_damper>
-                </ode>
-            </physics>
-        </joint>
-        <joint name="right_turnbuckle_joint" type="revolute">
-            <pose>-0.03 0 0 0 0 0</pose>
-            <axis>
-                <xyz>1 0 0</xyz>
-            </axis>
-            <parent>back_right_turnbuckle_link</parent>
-            <child>front_right_turnbuckle_link</child>
-            <physics>
-                <ode>
-                    <implicit_spring_damper>1</implicit_spring_damper>
-                </ode>
-            </physics>
-        </joint>
-    </gazebo>
+    <!-- Turnbuckle linkages between the differential and rockers
+        Note: URDF does not support closed loops in the robot description,
+        whereas SDF for Gazebo does.
+        These links and joints are for Gazebo only and close the kinematic chain
+        for the differential.
+    -->
+    <xacro:macro name="turnbuckle_assembly" params="lat_label reflect">
+        <gazebo>
+            <link name="${lat_label}_turnbuckle_link">
+                <pose>0.035 ${reflect * 0.17} 0.07 0 0 0</pose>
+                <visual name="${lat_label}_turnbuckle_visual">
+                    <pose>0 0 0 0 0 0</pose>
+                    <geometry>
+                        <mesh>
+                            <uri>package://curio_description/meshes/bases/turnbuckle.stl</uri>
+                        </mesh>
+                        <!-- <cylinder>
+                            <length>0.07</length>
+                            <radius>0.0025</radius>
+                        </cylinder> -->
+                    </geometry>
+                    <material>
+                        <script>
+                            <name>Gazebo/Blue</name>
+                        </script>
+                    </material>
+                </visual>
+                <collision name="${lat_label}_turnbuckle_collision">
+                    <pose>0 0 0 0 ${math_pi_over_2} 0</pose>
+                    <geometry>
+                        <cylinder>
+                            <length>0.07</length>
+                            <radius>0.0025</radius>
+                        </cylinder>
+                    </geometry>
+                </collision>
+                <inertial>
+                    <mass>0.01</mass>
+                    <inertia>
+                        <ixx>0.0001</ixx>
+                        <ixy>0</ixy>
+                        <ixz>0</ixz>
+                        <iyy>0.0001</iyy>
+                        <iyz>0</iyz>
+                        <izz>0.0001</izz>
+                    </inertia>
+                </inertial>
+            </link>
+            <joint name="back_${lat_label}_turnbuckle_joint" type="ball">
+                <pose>-0.035 0 0 0 0 0</pose>
+                <parent>diff_brace_link</parent>
+                <child>${lat_label}_turnbuckle_link</child>
+            </joint>
+            <joint name="front_${lat_label}_turnbuckle_joint" type="ball">
+                <pose>0.035 0 0 0 0 0</pose>
+                <parent>${lat_label}_rocker_link</parent>
+                <child>${lat_label}_turnbuckle_link</child>
+            </joint>
+        </gazebo>
+    </xacro:macro>
+    <xacro:turnbuckle_assembly lat_label="left" reflect="1"/>
+    <xacro:turnbuckle_assembly lat_label="right" reflect="-1"/>
     <!-- Rocker -->
     <xacro:macro name="rocker_link" params="lat_label reflect">
@@ -437,5 +299,5 @@
         </gazebo>
     </xacro:macro>
-    <!-- Fixed Rocker Joint  -->
+    <!-- Fixed Rocker Joint (for testing)  -->
     <!-- <xacro:macro name="rocker_joint" params="lat_label reflect">
         <joint name="${lat_label}_rocker_joint" type="fixed">
@@ -596,5 +458,5 @@
         </gazebo>
     </xacro:macro>
-    <!-- Fixed Bogie Joint  -->
+    <!-- Fixed Bogie Joint  (for testing) -->
     <!-- <xacro:macro name="bogie_joint" params="lat_label reflect">
         <joint name="${lat_label}_bogie_joint" type="fixed">

Commit message: Add mesh for laser scan assembly.
1. Add mesh for a custom mounting bracket and cowling for the RPLidar A1.
2. Update robot description to use new mesh file.

File: curio_description/urdf/curio.urdf.xacro (robot description, xacro)
@@ -526,4 +526,4 @@
     <!-- Laser Scan Sensor -->
     <xacro:laser_link />
-    <xacro:laser_joint x="0.145" y="0.07" z="0.055" />
+    <xacro:laser_joint x="0.152" y="0.078" z="0.050" />
 </robot>

File: curio_description/urdf/curio_laser.xacro (robot description, xacro)
@@ -37,7 +37,7 @@
                 <origin rpy="0 0 0" xyz="0 0 0" />
                 <geometry>
-                    <mesh filename="package://curio_description/meshes/sensors/rplidar_a1_low.stl" />
+                    <mesh filename="package://curio_description/meshes/sensors/rplidar_a1_assembly_low.stl" />
                 </geometry>
-                <material name="black" />
+                <material name="white" />
             </visual>
             <collision>
@@ -51,5 +51,5 @@
         </link>
         <gazebo reference="laser">
-            <material>Gazebo/Black</material>
+            <material>Gazebo/White</material>
             <sensor type="ray" name="laser_sensor">
                 <always_on>true</always_on>
