Commit message: Ensure robot hardware joint names are sync'd with driver servos.
1. Rename steering joints to be consistent across packages (replace 'corner' with 'steer')

File: curio_description/urdf/curio.urdf.xacro (robot description, xacro)
@@ -45,6 +45,6 @@
                 back_left_wheel_joint, back_right_wheel_joint
             Steer joints controlled by ackermann_drive_controller:
-                front_left_corner_joint, front_right_corner_joint,
-                back_left_corner_joint, back_right_corner_joint,
+                front_left_steer_joint, front_right_steer_joint,
+                back_left_steer_joint, back_right_steer_joint,
         -->
         <plugin name="gazebo_ros_control" filename="libgazebo_ros_control.so">
@@ -314,6 +314,6 @@
     <xacro:rocker_joint lat_label="left" reflect="1"/>
     <xacro:rocker_joint lat_label="right" reflect="-1"/>
-    <xacro:macro name="corner_link" params="lon_label lat_label reflect">
-        <link name="${lon_label}_${lat_label}_corner_link">
+    <xacro:macro name="steer_link" params="lon_label lat_label reflect">
+        <link name="${lon_label}_${lat_label}_steer_link">
             <visual>
                 <origin rpy="0 0 0" xyz="0 0 0" />
@@ -335,32 +335,32 @@
                 x="0.1" y="0.1" z="0.1" />
         </link>
-        <gazebo reference="${lon_label}_${lat_label}_corner_link">
+        <gazebo reference="${lon_label}_${lat_label}_steer_link">
             <material>Gazebo/DarkGray</material>
         </gazebo>
     </xacro:macro>
-    <xacro:corner_link lon_label="front" lat_label="left" reflect="1"/>
-    <xacro:corner_link lon_label="front" lat_label="right" reflect="-1"/>
-    <xacro:macro name="front_corner_joint" params="lat_label reflect">
-        <joint name="front_${lat_label}_corner_joint" type="continuous">
+    <xacro:steer_link lon_label="front" lat_label="left" reflect="1"/>
+    <xacro:steer_link lon_label="front" lat_label="right" reflect="-1"/>
+    <xacro:macro name="front_steer_joint" params="lat_label reflect">
+        <joint name="front_${lat_label}_steer_joint" type="continuous">
             <origin rpy="0 0 0" xyz="0.2116 ${reflect * 0.075} -0.0279"/>
             <axis xyz="0 0 1" />
             <parent link="${lat_label}_rocker_link" />
-            <child link="front_${lat_label}_corner_link" />
-        </joint>
-        <transmission name="front_${lat_label}_corner_transmission" >
+            <child link="front_${lat_label}_steer_link" />
+        </joint>
+        <transmission name="front_${lat_label}_steer_transmission" >
             <type>transmission_interface/SimpleTransmission</type>
-            <actuator name="front_${lat_label}_corner_actuator">
+            <actuator name="front_${lat_label}_steer_actuator">
                 <mechanicalReduction>1</mechanicalReduction>
             </actuator>
-            <joint name="front_${lat_label}_corner_joint">
+            <joint name="front_${lat_label}_steer_joint">
                 <hardwareInterface>hardware_interface/PositionJointInterface</hardwareInterface>
             </joint>
         </transmission>
-        <gazebo reference="front_${lat_label}_corner_joint">
+        <gazebo reference="front_${lat_label}_steer_joint">
             <provideFeedback>true</provideFeedback>
         </gazebo>
     </xacro:macro>
-    <xacro:front_corner_joint lat_label="left" reflect="1"/>
-    <xacro:front_corner_joint lat_label="right" reflect="-1"/>
+    <xacro:front_steer_joint lat_label="left" reflect="1"/>
+    <xacro:front_steer_joint lat_label="right" reflect="-1"/>
     <xacro:macro name="wheel_link" params="lon_label lat_label reflect">
         <link name="${lon_label}_${lat_label}_wheel_link">
@@ -389,9 +389,9 @@
     <xacro:wheel_link lon_label="front" lat_label="left" reflect="1"/>
     <xacro:wheel_link lon_label="front" lat_label="right" reflect="-1"/>
-    <xacro:macro name="corner_wheel_joint" params="lon_label lat_label reflect">
+    <xacro:macro name="steer_wheel_joint" params="lon_label lat_label reflect">
         <joint name="${lon_label}_${lat_label}_wheel_joint" type="continuous">
             <origin rpy="0 0 0" xyz="0 0 -0.132"/>
             <axis xyz="0 1 0" />
-            <parent link="${lon_label}_${lat_label}_corner_link" />
+            <parent link="${lon_label}_${lat_label}_steer_link" />
             <child link="${lon_label}_${lat_label}_wheel_link" />
         </joint>
@@ -409,6 +409,6 @@
         </gazebo>
     </xacro:macro>
-    <xacro:corner_wheel_joint lon_label="front" lat_label="left" reflect="1"/>
-    <xacro:corner_wheel_joint lon_label="front" lat_label="right" reflect="-1"/>
+    <xacro:steer_wheel_joint lon_label="front" lat_label="left" reflect="1"/>
+    <xacro:steer_wheel_joint lon_label="front" lat_label="right" reflect="-1"/>
     <!-- Bogie -->
     <xacro:macro name="bogie_link" params="lat_label reflect">
@@ -497,32 +497,32 @@
     <xacro:mid_wheel_joint lat_label="left" reflect="1"/>
     <xacro:mid_wheel_joint lat_label="right" reflect="-1"/>
-    <xacro:corner_link lon_label="back" lat_label="left" reflect="1"/>
-    <xacro:corner_link lon_label="back" lat_label="right" reflect="-1"/>
-    <xacro:macro name="back_corner_joint" params="lat_label reflect">
-        <joint name="back_${lat_label}_corner_joint" type="continuous">
+    <xacro:steer_link lon_label="back" lat_label="left" reflect="1"/>
+    <xacro:steer_link lon_label="back" lat_label="right" reflect="-1"/>
+    <xacro:macro name="back_steer_joint" params="lat_label reflect">
+        <joint name="back_${lat_label}_steer_joint" type="continuous">
             <origin rpy="0 0 0" xyz="-0.149 ${reflect * 0.05} 0.0338"/>
             <axis xyz="0 0 1" />
             <parent link="${lat_label}_bogie_link" />
-            <child link="back_${lat_label}_corner_link" />
-        </joint>
-        <transmission name="back_${lat_label}_corner_transmission" >
+            <child link="back_${lat_label}_steer_link" />
+        </joint>
+        <transmission name="back_${lat_label}_steer_transmission" >
             <type>transmission_interface/SimpleTransmission</type>
-            <actuator name="back_${lat_label}_corner_actuator">
+            <actuator name="back_${lat_label}_steer_actuator">
                 <mechanicalReduction>1</mechanicalReduction>
             </actuator>
-            <joint name="back_${lat_label}_corner_joint">
+            <joint name="back_${lat_label}_steer_joint">
                 <hardwareInterface>hardware_interface/PositionJointInterface</hardwareInterface>
             </joint>
         </transmission>
-        <gazebo reference="back_${lat_label}_corner_joint">
+        <gazebo reference="back_${lat_label}_steer_joint">
             <provideFeedback>true</provideFeedback>
         </gazebo>
     </xacro:macro>
-    <xacro:back_corner_joint lat_label="left" reflect="1"/>
-    <xacro:back_corner_joint lat_label="right" reflect="-1"/>
+    <xacro:back_steer_joint lat_label="left" reflect="1"/>
+    <xacro:back_steer_joint lat_label="right" reflect="-1"/>
     <xacro:wheel_link lon_label="back" lat_label="left" reflect="1"/>
     <xacro:wheel_link lon_label="back" lat_label="right" reflect="-1"/>
-    <xacro:corner_wheel_joint lon_label="back" lat_label="left" reflect="1"/>
-    <xacro:corner_wheel_joint lon_label="back" lat_label="right" reflect="-1"/>
+    <xacro:steer_wheel_joint lon_label="back" lat_label="left" reflect="1"/>
+    <xacro:steer_wheel_joint lon_label="back" lat_label="right" reflect="-1"/>
     <!-- IMU  -->
     <xacro:imu_link />
